Commit message: finished sensors

File: body.urdf (robot description, URDF)
Before this commit: robot robot, 3 links, 2 joints
Links:
- removed link Link0
- removed link Link1
- removed link Link2
- added link BackLeg, mass 1; collision box size=1 1 1; visual box size=1 1 1
- added link FrontLeg, mass 1; collision box size=1 1 1; visual box size=1 1 1
- added link Torso, mass 1; collision box size=1 1 1; visual box size=1 1 1
Joints:
- removed joint Link0_Link1
- removed joint Link1_Link2
- added joint BackLeg_Torso: type revolute, parent BackLeg, child Torso, origin xyz=1 0.5 1 rpy=0 0 0, axis 0 1 0, limit lower=-3.14159 upper=3.14159 effort=0.0 velocity=0.0
- added joint Torso_FrontLeg: type revolute, parent Torso, child FrontLeg, origin xyz=1 0 0 rpy=0 0 0, axis 0 1 0, limit lower=-3.14159 upper=3.14159 effort=0.0 velocity=0.0

Commit message: refactor body

File: body.urdf (robot description, URDF)
Before this commit: robot robot, 3 links, 2 joints
Joints:
- removed joint BackLeg_Torso
- added joint Torso_BackLeg: type revolute, parent Torso, child BackLeg, origin xyz=1 0.5 1 rpy=0 0 0, axis 0 1 0, limit lower=-3.14159 upper=3.14159 effort=0.0 velocity=0.0
- joint Torso_FrontLeg: origin xyz=1 0 0 rpy=0 0 0 -> xyz=2 0.5 1 rpy=0 0 0

Commit message: next: add lowers legs

File: body.urdf (robot description, URDF)
Before this commit: robot robot, 3 links, 2 joints
Links:
- added link LeftLeg, mass 1; collision box size=1 0.2 0.2; visual box size=1 0.2 0.2
- added link RightLeg, mass 1; collision box size=1 0.2 0.2; visual box size=1 0.2 0.2
- link BackLeg: geometry collision box size=0.2 1 0.2; visual box size=0.2 1 0.2
- link FrontLeg: geometry collision box size=0.2 1 0.2; visual box size=0.2 1 0.2
Joints:
- added joint Torso_LeftLeg: type revolute, parent Torso, child LeftLeg, origin xyz=-0.5 0 1 rpy=0 0 0, axis 1 0 0, limit lower=-3.14159 upper=3.14159 effort=0.0 velocity=0.0
- added joint Torso_RightLeg: type revolute, parent Torso, child RightLeg, origin xyz=0.5 0 1 rpy=0 0 0, axis 1 0 0, limit lower=-3.14159 upper=3.14159 effort=0.0 velocity=0.0
- joint Torso_BackLeg: axis 0 1 0 -> 1 0 0; origin xyz=1 0.5 1 rpy=0 0 0 -> xyz=0 -0.5 1 rpy=0 0 0
- joint Torso_FrontLeg: axis 0 1 0 -> 1 0 0; origin xyz=2 0.5 1 rpy=0 0 0 -> xyz=0 0.5 1 rpy=0 0 0

Commit message: deliverable 1

File: body.urdf (robot description, URDF)
Before this commit: robot robot, 9 links, 8 joints
Links:
- removed link BackLeg
- removed link BackLowerLeg
- removed link FrontLeg
- removed link FrontLowerLeg
- removed link LeftLeg
- removed link LeftLowerLeg
- removed link RightLeg
- removed link RightLowerLeg
- added link Arm, mass 1; collision box size=0.2 0.2 1; visual box size=0.2 0.2 1
- added link LegBackLeft, mass 1; collision box size=0.2 0.2 1; visual box size=0.2 0.2 1
- added link LegBackRight, mass 1; collision box size=0.2 0.2 1; visual box size=0.2 0.2 1
- added link LegFrontLeg, mass 1; collision box size=0.2 0.2 1; visual box size=0.2 0.2 1
- added link LegFrontRight, mass 1; collision box size=0.2 0.2 1; visual box size=0.2 0.2 1
- added link UpperArm, mass 1; collision box size=1 0.2 0.2; visual box size=1 0.2 0.2
- link Torso: geometry collision box size=2 1 1; visual box size=2 1 1
Joints:
- removed joint BackLeg_BackLowerLeg
- removed joint FrontLeg_FrontLowerLeg
- removed joint LeftLeg_LeftLowerLeg
- removed joint RightLeg_RightLowerLeg
- removed joint Torso_BackLeg
- removed joint Torso_FrontLeg
- removed joint Torso_LeftLeg
- removed joint Torso_RightLeg
- added joint Arm_UpperArm: type revolute, parent Arm, child UpperArm, origin xyz=0 0 1 rpy=0 0 0, axis 0 1 0, limit lower=-3.14159 upper=3.14159 effort=0.0 velocity=0.0
- added joint Torso_Arm: type revolute, parent Torso, child Arm, origin xyz=-1 0 2 rpy=0 0 0, axis 0 1 0, limit lower=-3.14159 upper=3.14159 effort=0.0 velocity=0.0
- added joint Torso_LegBackLeft: type revolute, parent Torso, child LegBackLeft, origin xyz=1 -0.5 1 rpy=0 0 0, axis 0 1 0, limit lower=-3.14159 upper=3.14159 effort=0.0 velocity=0.0
- added joint Torso_LegBackRight: type revolute, parent Torso, child LegBackRight, origin xyz=1 0.5 1 rpy=0 0 0, axis 0 1 0, limit lower=-3.14159 upper=3.14159 effort=0.0 velocity=0.0
- added joint Torso_LegFrontLeft: type revolute, parent Torso, child LegFrontLeg, origin xyz=-1 -0.5 1 rpy=0 0 0, axis 0 1 0, limit lower=-3.14159 upper=3.14159 effort=0.0 velocity=0.0
- added joint Torso_LegFrontRight: type revolute, parent Torso, child LegFrontRight, origin xyz=-1 0.5 1 rpy=0 0 0, axis 0 1 0, limit lower=-3.14159 upper=3.14159 effort=0.0 velocity=0.0
